File: CH7800_EK.kicad_pcb (KiCad board)
At the start: 2 copper layers, 65 x 40 mm, 20 parts, among them J1 USB_C_Receptacle_USB2.0_16P, J2 Conn_01x02_Pin, J3 Conn_01x07_Pin, U1 USBLC6-2SC6, U2 CH7800

Commit message: v1.1 with production file
Parts:
- moved R1 1.33 mm to (100.5, 111.5)
- moved R2 1.33 mm to (100.5, 114.0)
- moved J2 1.00 mm to (110.0, 88.5)
- moved J3 1.00 mm to (117.3, 88.5)
- moved Speaker1 1.00 mm to (154.5, 106.8)
Routing:
- net Net-(J1-CC2): track 14.5 -> 11.9 mm
- net Net-(J1-CC1): track 14.4 -> 12.9 mm
- net /SPK+: track 30.3 -> 28.9 mm
- net /tx: track 14.8 -> 13.8 mm
- net /rx: track 14.8 -> 13.8 mm
- net /dac: track 15.3 -> 14.3 mm
- net VCC: track 35.9 -> 34.9 mm
- net /busy: track 20.9 -> 19.9 mm
- net /SPK-: track 28.0 -> 27.0 mm
- net +3.3V: track 25.2 -> 24.2 mm
- net VBUS: track 38.1 -> 37.1 mm
Other:
- board text added: "I/O"
- board text added: "PPK2"
- board text removed: "V_{in}"
- board text removed: "V_{out}"
